Commit message: change to lesson3

File: robot/summit.urdf.xacro (robot description, xacro)
@@ -10,16 +10,17 @@
 	<xacro:macro name="robot">
 		<xacro:summit_base/>
-		<xacro:omni_wheel prefix="summit_front_right" parent="summit_base_footprint" reflect="false">
+		<xacro:omni_wheel prefix="summit_front_right" parent="summit_base_link" reflect="false">
 			<origin xyz="${wheel_offset_x} -${wheel_offset_y} ${wheel_offset_z}" rpy="0 0 0"/>
 		</xacro:omni_wheel>
-		<xacro:omni_wheel prefix="summit_front_left" parent="summit_base_footprint" reflect="true">
+		<xacro:omni_wheel prefix="summit_front_left" parent="summit_base_link" reflect="true">
 			<origin xyz="${wheel_offset_x} ${wheel_offset_y} ${wheel_offset_z}" rpy="0 0 0"/>
 		</xacro:omni_wheel>
-		<xacro:omni_wheel prefix="summit_back_left" parent="summit_base_footprint" reflect="true">
+		<xacro:omni_wheel prefix="summit_back_left" parent="summit_base_link" reflect="true">
 			<origin xyz="-${wheel_offset_x} ${wheel_offset_y} ${wheel_offset_z}" rpy="0 0 0"/>
 		</xacro:omni_wheel>
-		<xacro:omni_wheel prefix="summit_back_right" parent="summit_base_footprint" reflect="false">
+		<xacro:omni_wheel prefix="summit_back_right" parent="summit_base_link" reflect="false">
 			<origin xyz="-${wheel_offset_x} -${wheel_offset_y} ${wheel_offset_z}" rpy="0 0 0"/>
 		</xacro:omni_wheel>
+        <xacro:omni_steering/>
    </xacro:macro>
    <xacro:robot/>

File: urdf/base/summit_base.urdf.xacro (robot description, xacro)
@@ -2,4 +2,5 @@
 <robot name="summit_xl" xmlns:xacro="http://www.ros.org/wiki/xacro">
   <xacro:macro name="summit_base">
+      <xacro:include filename="$(find summit_description)/urdf/base/summit_base.gazebo.xacro" />
 	  <!-- Robot mechanical and motor parameters -->
 	  <xacro:property name="PI" value="3.1415926535897931"/>
@@ -13,10 +14,33 @@
 			  </geometry>
 		  </visual>
-          <inertial>
-            <mass value="125.0" />
-            <origin xyz="0 0 0" />
-            <inertia  ixx="1.391" ixy="0.004"  ixz="0.0"  iyy="6.853"  iyz="0.0"  izz="6.125" />
-        </inertial>
 		</link>
+		<joint name="summit_base_footprint_joint" type="fixed">
+		  <origin xyz="0 0 ${wheel_radius}" rpy="0 0 0" /> <!-- ${wheel_radius} property must be defined inside wheel description -->
+		  <parent link="summit_base_footprint"/>
+		  <child link="summit_base_link" />
+		</joint>
+  <!-- BASE_LINK -->
+  <link name="summit_base_link">
+    <inertial>
+      <mass value="125.0" />
+      <origin xyz="0 0 0" />
+      <inertia  ixx="1.391" ixy="0.004"  ixz="0.0"  iyy="6.853"  iyz="0.0"  izz="6.125" />
+    </inertial>
+    <visual>
+       <origin xyz="0 0 0" rpy="0 0 0" />
+       <geometry>
+	     <mesh filename="package://summit_description/meshes/base/summit_base.dae"/>
+       </geometry>
+       <material name="darkgrey">
+         <color rgba="0.1 0.1 0.1 1"/>
+       </material>
+    </visual>
+    <collision>
+       <origin xyz="0 0 0" rpy="0 0 0 " />
+       <geometry>
+         <mesh filename="package://summit_description/meshes/base/summit_base.dae"/>
+       </geometry>
+    </collision>
+  </link>
   </xacro:macro>
 </robot>

File: urdf/wheels/omni_wheel.urdf.xacro (robot description, xacro)
@@ -1,10 +1,9 @@
 <?xml version="1.0"?>
 <robot name="wheel" xmlns:xacro="http://www.ros.org/wiki/xacro">
-  <!-- Constants -->
   <xacro:property name="PI" value="3.1415926535897931" />
+  <!-- Wheels -->
   <xacro:property name="wheel_radius" value="0.127" />
   <xacro:property name="wheel_height" value="0.087" />
   <xacro:property name="wheel_mass" value="6.5" /> <!-- in kg-->
-  <!-- Simple Macro to calculate inertia -->
   <xacro:macro name="cylinder_inertia" params="m r h">
     <inertia  ixx="${m*(3*r*r+h*h)/12}" ixy = "0" ixz = "0"
@@ -12,6 +11,13 @@
               izz="${m*(3*r*r+h*h)/12}" />
   </xacro:macro>
-  <!-- Set up of the Wheel -->
   <xacro:macro name="omni_wheel" params="prefix parent *origin reflect">
+    <joint name="${prefix}_wheel_joint" type="continuous">
+      <parent link="${parent}"/>
+      <child link="${prefix}_wheel_link"/>
+      <xacro:insert_block name="origin" />
+      <axis xyz="0 1 0" rpy="0 0 0" />
+      <limit effort="100" velocity="100"/>
+      <joint_properties damping="0.0" friction="0.0"/>
+    </joint>
     <link name="${prefix}_wheel_link">
       <visual>
@@ -40,12 +46,4 @@
       </inertial>
     </link>
-    <joint name="${prefix}_wheel_joint" type="continuous">
-      <parent link="${parent}"/>
-      <child link="${prefix}_wheel_link"/>
-      <xacro:insert_block name="origin" />
-      <axis xyz="0 1 0" rpy="0 0 0" />
-      <limit effort="100" velocity="100"/>
-      <joint_properties damping="0.0" friction="0.0"/>
-    </joint>
     <!-- Transmission is important to link the joints and the controller (see summit_xl_control/config/summit_xl_control.yaml)-->
     <transmission name="${prefix}_wheel_joint_trans">
